File: pcb/smart_smartyKat_crazy_cruiser.kicad_sch (KiCad schematic)
At the start: 12 parts, among them M1 Vibe, Q1 NCE3401, Q2 NCE3401, SW1 Power, SW2 SW-18001P, U1 PFS154-S08

Commit message: simplify schema
Parts:
- removed C1: 100n, symbol Device:C
- removed D3: D, symbol Device:D
- removed R2: 10k, symbol Device:R
Connections:
- net GND: now also R1.2; no longer D2.1 (K)
- net LED: now also D2.2 (A); no longer R1.1
- new net: D2.1 (K), R1.1
Other:
- moved on the sheet: D2, R1
Changed lines of the file:
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@@
   (title_block
     (title "Smart Mod for SmartyKat Crazy Cruiser")
-    (date "2023-02-11")
+    (date "2023-03-04")
     (company "erry Leuams")
   )
-  (junction (at 184.15 81.28) (diameter 0) (color 0 0 0 0)
-  )
-  (junction (at 173.99 93.98) (diameter 0) (color 0 0 0 0)
-  )
   (junction (at 121.92 80.01) (diameter 0) (color 0 0 0 0)
-  )
-  (junction (at 184.15 116.84) (diameter 0) (color 0 0 0 0)
-  )
-  (junction (at 144.78 88.9) (diameter 0) (color 0 0 0 0)
-  )
-  (junction (at 184.15 101.6) (diameter 0) (color 0 0 0 0)
   )
   (no_connect (at 124.46 93.98))
@@
   (no_connect (at 124.46 96.52))
   (no_connect (at 102.87 85.09))
-  (wire (pts (xy 184.15 116.84) (xy 184.15 118.11))
+  (wire (pts (xy 184.15 115.57) (xy 184.15 118.11))
     (stroke (width 0) (type default) (color 0 0 0 0))
   )
@@
     (stroke (width 0) (type default) (color 0 0 0 0))
   )
-  (wire (pts (xy 173.99 81.28) (xy 184.15 81.28))
-    (stroke (width 0) (type default) (color 0 0 0 0))
-  )
   (wire (pts (xy 82.55 82.55) (xy 92.71 82.55))
     (stroke (width 0) (type default) (color 0 0 0 0))
@@
     (stroke (width 0) (type default) (color 0 0 0 0))
   )
-  (wire (pts (xy 173.99 85.09) (xy 173.99 81.28))
-    (stroke (width 0) (type default) (color 0 0 0 0))
-  )
   (wire (pts (xy 121.92 76.2) (xy 121.92 80.01))
     (stroke (width 0) (type default) (color 0 0 0 0))
@@
     (stroke (width 0) (type default) (color 0 0 0 0))
   )
-  (wire (pts (xy 129.54 80.01) (xy 121.92 80.01))
-    (stroke (width 0) (type default) (color 0 0 0 0))
-  )
   (wire (pts (xy 121.92 88.9) (xy 124.46 88.9))
     (stroke (width 0) (type default) (color 0 0 0 0))
@@
     (stroke (width 0) (type default) (color 0 0 0 0))
   )
-  (wire (pts (xy 184.15 116.84) (xy 194.31 116.84))
-    (stroke (width 0) (type default) (color 0 0 0 0))
-  )
   (wire (pts (xy 170.18 105.41) (xy 170.18 107.95))
     (stroke (width 0) (type default) (color 0 0 0 0))
   )
-  (wire (pts (xy 184.15 81.28) (xy 184.15 88.9))
-    (stroke (width 0) (type default) (color 0 0 0 0))
-  )
-  (wire (pts (xy 184.15 101.6) (xy 184.15 102.87))
-    (stroke (width 0) (type default) (color 0 0 0 0))
-  )
-  (wire (pts (xy 137.16 80.01) (xy 144.78 80.01))
-    (stroke (width 0) (type default) (color 0 0 0 0))
-  )
-  (wire (pts (xy 173.99 93.98) (xy 176.53 93.98))
-    (stroke (width 0) (type default) (color 0 0 0 0))
-  )
-  (wire (pts (xy 144.78 80.01) (xy 144.78 88.9))
+  (wire (pts (xy 184.15 80.01) (xy 184.15 88.9))
+    (stroke (width 0) (type default) (color 0 0 0 0))
+  )
+  (wire (pts (xy 184.15 99.06) (xy 184.15 102.87))
+    (stroke (width 0) (type default) (color 0 0 0 0))
+  )
+  (wire (pts (xy 142.24 93.98) (xy 176.53 93.98))
     (stroke (width 0) (type default) (color 0 0 0 0))
   )
@@
     (stroke (width 0) (type default) (color 0 0 0 0))
   )
-  (wire (pts (xy 184.15 99.06) (xy 184.15 101.6))
-    (stroke (width 0) (type default) (color 0 0 0 0))
-  )
-  (wire (pts (xy 142.24 93.98) (xy 173.99 93.98))
-    (stroke (width 0) (type default) (color 0 0 0 0))
-  )
   (wire (pts (xy 151.13 82.55) (xy 148.59 82.55))
     (stroke (width 0) (type default) (color 0 0 0 0))
   )
-  (wire (pts (xy 194.31 105.41) (xy 194.31 101.6))
-    (stroke (width 0) (type default) (color 0 0 0 0))
-  )
   (wire (pts (xy 144.78 88.9) (xy 144.78 101.6))
     (stroke (width 0) (type default) (color 0 0 0 0))
   )
-  (wire (pts (xy 194.31 101.6) (xy 184.15 101.6))
-    (stroke (width 0) (type default) (color 0 0 0 0))
-  )
-  (wire (pts (xy 184.15 80.01) (xy 184.15 81.28))
-    (stroke (width 0) (type default) (color 0 0 0 0))
-  )
-  (wire (pts (xy 173.99 92.71) (xy 173.99 93.98))
-    (stroke (width 0) (type default) (color 0 0 0 0))
-  )
-  (wire (pts (xy 194.31 113.03) (xy 194.31 116.84))
-    (stroke (width 0) (type default) (color 0 0 0 0))
-  )
   (wire (pts (xy 160.02 105.41) (xy 157.48 105.41))
-    (stroke (width 0) (type default) (color 0 0 0 0))
-  )
-  (wire (pts (xy 184.15 115.57) (xy 184.15 116.84))
     (stroke (width 0) (type default) (color 0 0 0 0))
   )
@@
     (effects (font (size 1.27 1.27)) (justify left bottom))
   )
-  (symbol (lib_id "Device:LED") (at 163.83 105.41 0) (mirror y) (unit 1)
-    (in_bom yes) (on_board yes)
-    (property "Reference" "D2" (id 0) (at 163.83 102.87 0))
-    (property "Value" "YLW" (id 1) (at 163.83 107.95 0))
-    (property "Footprint" "" (id 2) (at 163.83 105.41 0)
-      (effects (font (size 1.27 1.27)) hide)
-    )
-    (property "Datasheet" "~" (id 3) (at 163.83 105.41 0)
+  (symbol (lib_id "Device:LED") (at 153.67 105.41 0) (mirror y) (unit 1)
+    (in_bom yes) (on_board yes)
+    (property "Reference" "D2" (id 0) (at 153.67 102.87 0))
+    (property "Value" "YLW" (id 1) (at 153.67 107.95 0))
+    (property "Footprint" "" (id 2) (at 153.67 105.41 0)
+      (effects (font (size 1.27 1.27)) hide)
+    )
+    (property "Datasheet" "~" (id 3) (at 153.67 105.41 0)
       (effects (font (size 1.27 1.27)) hide)
     )
@@
     )
     (pin "1")
-  )
-  (symbol (lib_id "Device:D") (at 194.31 109.22 270) (unit 1)
-    (in_bom yes) (on_board yes)
-    (property "Reference" "D3" (id 0) (at 196.85 109.22 0))
-    (property "Value" "D" (id 1) (at 191.77 109.22 0))
-    (property "Footprint" "" (id 2) (at 194.31 109.22 0)
-      (effects (font (size 1.27 1.27)) hide)
-    )
-    (property "Datasheet" "~" (id 3) (at 194.31 109.22 0)
-      (effects (font (size 1.27 1.27)) hide)
-    )
-    (pin "1")
-    (pin "2")
-  )
-  (symbol (lib_id "Device:R") (at 173.99 88.9 180) (unit 1)
-    (in_bom yes) (on_board yes)
-    (property "Reference" "R2" (id 0) (at 171.958 88.9 90))
-    (property "Value" "10k" (id 1) (at 173.99 88.9 90))
-    (property "Footprint" "" (id 2) (at 175.768 88.9 90)
-      (effects (font (size 1.27 1.27)) hide)
-    )
-    (property "Datasheet" "~" (id 3) (at 173.99 88.9 0)
-      (effects (font (size 1.27 1.27)) hide)
-    )
-    (pin "1")
-    (pin "2")
   )
   (symbol (lib_id "Device:Q_PMOS_GSD") (at 110.49 82.55 90) (unit 1)
@@
     (pin "1")
   )
-  (symbol (lib_id "Device:C") (at 133.35 80.01 90) (unit 1)
-    (in_bom yes) (on_board yes)
-    (property "Reference" "C1" (id 0) (at 130.81 79.375 0)
-      (effects (font (size 1.27 1.27)) (justify left))
-    )
-    (property "Value" "100n" (id 1) (at 135.89 79.375 0)
-      (effects (font (size 1.27 1.27)) (justify left))
-    )
-    (property "Footprint" "" (id 2) (at 137.16 79.0448 0)
-      (effects (font (size 1.27 1.27)) hide)
-    )
-    (property "Datasheet" "~" (id 3) (at 133.35 80.01 0)
-      (effects (font (size 1.27 1.27)) hide)
-    )
-    (pin "1")
-    (pin "2")
-  )
-  (symbol (lib_id "Device:R") (at 153.67 105.41 90) (mirror x) (unit 1)
-    (in_bom yes) (on_board yes)
-    (property "Reference" "R1" (id 0) (at 153.67 107.442 90))
-    (property "Value" "100" (id 1) (at 153.67 105.41 90))
-    (property "Footprint" "" (id 2) (at 153.67 103.632 90)
-      (effects (font (size 1.27 1.27)) hide)
-    )
-    (property "Datasheet" "~" (id 3) (at 153.67 105.41 0)
+  (symbol (lib_id "Device:R") (at 163.83 105.41 90) (mirror x) (unit 1)
+    (in_bom yes) (on_board yes)
+    (property "Reference" "R1" (id 0) (at 163.83 107.442 90))
+    (property "Value" "100" (id 1) (at 163.83 105.41 90))
+    (property "Footprint" "" (id 2) (at 163.83 103.632 90)
+      (effects (font (size 1.27 1.27)) hide)
+    )
+    (property "Datasheet" "~" (id 3) (at 163.83 105.41 0)
       (effects (font (size 1.27 1.27)) hide)
     )
@@
       (reference "BT1") (unit 1) (value "2x LR44") (footprint "")
     )
-    (path "/e9c31c2e-fd01-4189-bd1c-7e08ccbc54e8"
-      (reference "C1") (unit 1) (value "100n") (footprint "")
-    )
     (path "/03c0d40b-d85b-4216-b77e-379e8408b7fe"
       (reference "D2") (unit 1) (value "YLW") (footprint "")
     )
-    (path "/775e3280-3099-44e0-9035-a355a5874275"
-      (reference "D3") (unit 1) (value "D") (footprint "")
-    )
     (path "/db780385-0091-42be-9e12-708823263557"
       (reference "M1") (unit 1) (value "Vibe") (footprint "")
@@
       (reference "R1") (unit 1) (value "100") (footprint "")
     )
-    (path "/8a4f39d5-6438-4dde-9278-c37b6854559e"
-      (reference "R2") (unit 1) (value "10k") (footprint "")
-    )
     (path "/6542813c-dbe4-4109-a9c2-a70b34d8fe28"
